File: hardware/midiwall.brd (EAGLE design)
At the start: 80.6 x 34.9 mm, 29 parts, among them IC1 PIC12F1822SO08

Commit message: v2 poss
Routing:
- net KEY2: track 65.5 -> 69.6 mm
- net N$5: track 19.2 -> 20.4 mm
- net N$9: track 20.1 -> 20.7 mm
Other:
- board size 80.6 x 34.9 mm -> 80.7 x 36.8 mm
- board text added: "MIDIWALL v2"
- board text removed: "MIDIWALL v1"
Changed lines of the file:
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@@
 <board>
 <plain>
-<hole x="3.81" y="4.445" drill="3.2"/>
-<hole x="78.105" y="4.445" drill="3.2"/>
+<hole x="3.81" y="2.54" drill="3.2"/>
+<hole x="78.105" y="2.54" drill="3.2"/>
 <hole x="78.105" y="33.02" drill="3.2"/>
 <hole x="3.81" y="33.02" drill="3.2"/>
@@
 <wire x1="3.175" y1="36.195" x2="78.74" y2="36.195" width="0.4064" layer="20"/>
 <wire x1="78.74" y1="36.195" x2="81.28" y2="33.655" width="0.4064" layer="20" curve="-90"/>
-<wire x1="81.28" y1="33.655" x2="81.28" y2="3.81" width="0.4064" layer="20"/>
-<wire x1="81.28" y1="3.81" x2="78.74" y2="1.27" width="0.4064" layer="20" curve="-90"/>
-<wire x1="78.74" y1="1.27" x2="3.175" y2="1.27" width="0.4064" layer="20"/>
-<wire x1="3.175" y1="1.27" x2="0.635" y2="3.81" width="0.4064" layer="20" curve="-90"/>
-<wire x1="0.635" y1="3.81" x2="0.635" y2="33.655" width="0.4064" layer="20"/>
-<text x="9.017" y="32.893" size="2.54" layer="25" font="vector" ratio="20">MIDIWALL v1</text>
-<text x="59.055" y="33.655" size="1.778" layer="25" font="vector" ratio="20">hotchk155</text>
+<wire x1="81.28" y1="33.655" x2="81.28" y2="2.54" width="0.4064" layer="20"/>
+<wire x1="81.28" y1="2.54" x2="78.74" y2="-0.635" width="0.4064" layer="20" curve="-90"/>
+<wire x1="78.74" y1="-0.635" x2="3.175" y2="-0.635" width="0.4064" layer="20"/>
+<wire x1="3.175" y1="-0.635" x2="0.635" y2="2.54" width="0.4064" layer="20" curve="-90"/>
+<wire x1="0.635" y1="2.54" x2="0.635" y2="33.655" width="0.4064" layer="20"/>
+<text x="9.017" y="32.893" size="2.54" layer="25" font="vector" ratio="20">MIDIWALL v2</text>
+<text x="61.595" y="0.635" size="1.778" layer="25" font="vector" ratio="20">hotchk155</text>
 </plain>
 <attributes>
@@
 </element>
 <element name="D6" library="jasons_stuff" package="0805DIODE" value="0805DIODE" x="50.165" y="10.16" smashed="yes" rot="R180">
-<attribute name="NAME" x="51.4428" y="12.489" size="1.27" layer="21" font="vector" ratio="20" rot="R180"/>
+<attribute name="NAME" x="51.4428" y="8.679" size="1.27" layer="21" font="vector" ratio="20" rot="R180"/>
 </element>
 <element name="D2" library="jasons_stuff" package="0805DIODE" value="0805DIODE" x="31.115" y="15.24" smashed="yes">
@@
 </element>
 <element name="D7" library="jasons_stuff" package="0805DIODE" value="0805DIODE" x="50.165" y="5.08" smashed="yes" rot="R180">
-<attribute name="NAME" x="51.5698" y="7.663" size="1.27" layer="21" font="vector" ratio="20" rot="R180"/>
+<attribute name="NAME" x="51.5698" y="3.853" size="1.27" layer="21" font="vector" ratio="20" rot="R180"/>
 </element>
 <element name="D5" library="jasons_stuff" package="0805DIODE" value="0805DIODE" x="50.165" y="15.24" smashed="yes" rot="R180">
@@
 </element>
 <element name="D1" library="jasons_stuff" package="0805DIODE" value="0805DIODE" x="31.115" y="20.32" smashed="yes">
-<attribute name="NAME" x="28.8212" y="17.737" size="1.27" layer="21" font="vector" ratio="20"/>
+<attribute name="NAME" x="27.5512" y="17.737" size="1.27" layer="21" font="vector" ratio="20"/>
 </element>
 <element name="D4" library="jasons_stuff" package="0805DIODE" value="0805DIODE" x="31.115" y="5.08" smashed="yes">
@@
 <wire x1="65.532" y1="28.829" x2="64.008" y2="28.829" width="0.3048" layer="16"/>
 <via x="64.008" y="28.829" extent="1-16" drill="0.6"/>
-<wire x1="69.469" y1="28.321" x2="69.469" y2="23.495" width="0.3048" layer="1"/>
-<wire x1="69.469" y1="23.495" x2="67.945" y2="21.971" width="0.3048" layer="1"/>
-<wire x1="67.945" y1="21.971" x2="67.945" y2="13.97" width="0.3048" layer="1"/>
+<wire x1="69.469" y1="28.321" x2="69.469" y2="24.765" width="0.3048" layer="1"/>
+<wire x1="69.469" y1="24.765" x2="67.945" y2="23.241" width="0.3048" layer="1"/>
+<wire x1="67.945" y1="23.241" x2="67.945" y2="13.97" width="0.3048" layer="1"/>
 <wire x1="67.945" y1="13.97" x2="69.088" y2="12.827" width="0.3048" layer="1"/>
 <wire x1="69.088" y1="12.827" x2="69.088" y2="10.16" width="0.3048" layer="1"/>
@@
 <wire x1="56.134" y1="32.004" x2="56.515" y2="32.385" width="0.3048" layer="1"/>
 <wire x1="56.515" y1="32.385" x2="61.722" y2="32.385" width="0.3048" layer="1"/>
-<wire x1="63.627" y1="13.589" x2="52.959" y2="2.921" width="0.3048" layer="1"/>
-<wire x1="52.959" y1="2.921" x2="49.784" y2="2.921" width="0.3048" layer="1"/>
 <wire x1="49.784" y1="2.921" x2="48.895" y2="3.81" width="0.3048" layer="1"/>
 <wire x1="48.895" y1="3.81" x2="48.895" y2="5.0532" width="0.3048" layer="1"/>
@@
 <wire x1="61.722" y1="32.385" x2="61.849" y2="32.258" width="0.3048" layer="1"/>
 <wire x1="61.849" y1="32.258" x2="61.849" y2="28.575" width="0.3048" layer="1"/>
-<wire x1="63.627" y1="26.797" x2="63.627" y2="13.589" width="0.3048" layer="1"/>
 <wire x1="61.849" y1="28.575" x2="63.627" y2="26.797" width="0.3048" layer="1"/>
+<wire x1="63.627" y1="26.797" x2="63.627" y2="16.637" width="0.3048" layer="1"/>
+<wire x1="63.627" y1="16.637" x2="62.23" y2="15.24" width="0.3048" layer="1"/>
+<wire x1="62.23" y1="15.24" x2="62.23" y2="5.08" width="0.3048" layer="1"/>
+<wire x1="62.23" y1="5.08" x2="61.595" y2="4.445" width="0.3048" layer="1"/>
+<wire x1="61.595" y1="4.445" x2="60.96" y2="3.81" width="0.3048" layer="1"/>
+<wire x1="49.784" y1="2.921" x2="60.071" y2="2.921" width="0.3048" layer="1"/>
+<wire x1="60.071" y1="2.921" x2="60.96" y2="3.81" width="0.3048" layer="1"/>
 </signal>
 <signal name="+5V">
@@
 <contactref element="R7" pad="1"/>
 <contactref element="R9" pad="2"/>
-<wire x1="71.12" y1="24.45" x2="71.12" y2="21.995" width="0.3048" layer="1"/>
-<wire x1="71.12" y1="21.995" x2="70.105" y2="20.98" width="0.3048" layer="1"/>
-<wire x1="71.12" y1="11.11" x2="71.12" y2="11.43" width="0.3048" layer="1"/>
 <wire x1="71.12" y1="11.43" x2="74.93" y2="15.24" width="0.3048" layer="1"/>
-<wire x1="74.93" y1="15.24" x2="74.93" y2="20.32" width="0.3048" layer="1"/>
-<wire x1="71.12" y1="21.995" x2="73.255" y2="21.995" width="0.3048" layer="1"/>
-<wire x1="73.255" y1="21.995" x2="74.93" y2="20.32" width="0.3048" layer="1"/>
+<wire x1="74.93" y1="15.24" x2="74.93" y2="20.64" width="0.3048" layer="1"/>
+<wire x1="74.93" y1="20.64" x2="71.12" y2="24.45" width="0.3048" layer="1"/>
+<wire x1="71.12" y1="11.43" x2="71.12" y2="11.11" width="0.3048" layer="1"/>
+<wire x1="70.105" y1="14.63" x2="70.105" y2="12.125" width="0.3048" layer="1"/>
+<wire x1="70.105" y1="12.125" x2="71.12" y2="11.11" width="0.3048" layer="1"/>
 </signal>
 <signal name="N$8">
@@
 <wire x1="7.62" y1="15.24" x2="11.43" y2="11.43" width="0.3048" layer="1"/>
 <wire x1="11.43" y1="11.43" x2="11.43" y2="11.11" width="0.3048" layer="1"/>
-<wire x1="11.81" y1="14.58" x2="11.81" y2="11.49" width="0.3048" layer="1"/>
 <wire x1="11.81" y1="11.49" x2="11.43" y2="11.11" width="0.3048" layer="1"/>
 <wire x1="7.62" y1="15.24" x2="7.62" y2="20.32" width="0.3048" layer="1"/>
 <wire x1="7.62" y1="20.32" x2="11.43" y2="24.13" width="0.3048" layer="1"/>
 <wire x1="11.43" y1="24.13" x2="11.43" y2="24.45" width="0.3048" layer="1"/>
+<wire x1="11.81" y1="20.93" x2="11.81" y2="24.07" width="0.3048" layer="1"/>
+<wire x1="11.81" y1="24.07" x2="11.43" y2="24.45" width="0.3048" layer="1"/>
 </signal>
 <signal name="N$10">

Commit message: new case
Parts:
- R5: value (none) -> 4k7
Changed lines of the file:
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@@
 <attribute name="VALUE" x="77.47" y="9.525" size="1.27" layer="27" rot="R90"/>
 </element>
-<element name="R5" library="rcl" package="R0805" value="" x="59.055" y="30.226" smashed="yes">
+<element name="R5" library="rcl" package="R0805" value="4k7" x="59.055" y="30.226" smashed="yes">
 <attribute name="NAME" x="62.611" y="29.21" size="1.27" layer="25" font="vector" ratio="20" rot="R90"/>
 <attribute name="VALUE" x="58.42" y="27.686" size="1.27" layer="27"/>

Commit message: REV3
Parts:
- removed D2, D3, D4, D5, D6, D7: 0805DIODE, jasons_stuff:0805DIODE
- removed J1: (no value), tag-connect:TC2030-MCP-NL
- added ICSP: (no value), tag-connect:TC2030-MCP-NL
- added LED2: (no value), led:LED3MM
- added R11: (no value), rcl:R0805
- C1: device microbuilder:EIA3216-18/A-R -> rcl:E2,5-5
- IC1: value PIC12F1822SO08 -> PIC16F1825SO14; device jasons_stuff:SO08 -> jasons_stuff:SO14
- moved R5 52.4 mm to (6.99, 24.5)
- moved C2 22.0 mm to (70.0, 33.8), turned to 0 degrees
- moved C1 21.1 mm to (52.1, 30.5), turned to 90 degrees
- moved R8 18.6 mm to (69.6, 7.62), turned to 270 degrees
- moved D1 16.6 mm to (31.2, 3.68), turned to 270 degrees
- moved R2 16.1 mm to (6.10, 10.2)
- moved R1 15.8 mm to (3.30, 10.2)
- moved IC1 15.6 mm to (69.8, 27.9), turned to 270 degrees
- moved R7 10.9 mm to (61.0, 29.2), turned to 0 degrees
- moved R6 10.7 mm to (61.0, 32.0)
- moved LED1 3.17 mm to (56.5, 25.4), turned to 270 degrees
- moved R9 2.96 mm to (72.6, 7.62), turned to 270 degrees
- moved R10 2.65 mm to (75.7, 7.62)
- moved R3 1.27 mm to (8.89, 10.2), turned to 90 degrees
- moved R4 0.25 mm to (11.7, 10.2), turned to 90 degrees
Connections:
- removed net KEY0: D5.C, D6.C, IC1.4, J1.1
- removed net N$10: LED1.K, R6.2
- removed net N$11: IC1.2, LED1.A
- removed net N$3: D7.A, SW4.3, SW4.4
- removed net N$4: D1.A, D5.A, SW2.3, SW2.4
- removed net N$6: D3.A, D4.A, SW3.3, SW3.4
- new net KEY3: IC1.11, SW4.3, SW4.4
- new net KEY4: IC1.8, SW1.3, SW1.4
- new net KEY5: IC1.10, SW5.3, SW5.4
- new net LED1: IC1.2, R6.2
- new net LED2: IC1.3, R7.2
- new net PGC: IC1.12, ICSP.5
- new net PGD: IC1.13, ICSP.4
- new net VPP: IC1.4, ICSP.1
- net +5V: now also D1.A, ICSP.2, R10.2, R11.2; no longer J1.2, R7.2, R8.2
- net GND: now also D1.C, IC1.14, ICSP.3, LED1.K, LED2.K; no longer IC1.8, J1.3, R6.1
- net KEY1: now also IC1.9, SW3.3, SW3.4; no longer D1.C, D2.C, D3.C, IC1.3
- net KEY2: now also IC1.7, SW2.3, SW2.4; no longer D4.C, D7.C, IC1.5
- net N$1: now also LED1.A, R6.1; no longer D6.A, SW5.3, SW5.4
- net N$2: now also LED2.A, R7.1; no longer D2.A, SW1.3, SW1.4
- net N$5: now also R11.1, R8.2; no longer R7.1, R9.2
- net N$7: now also R4.1; no longer R3.1
- net N$8: now also R10.1, R9.2; no longer R10.2, R8.1
- net N$9: now also R3.1; no longer R4.1
- net RX: now also IC1.5; no longer IC1.6, J1.5
- net TX: now also IC1.6, R8.1; no longer IC1.7, J1.4, R10.1
Routing:
- net KEY4: track 0.00 -> 64.1 mm, vias 0 -> 1
- net KEY3: track 0.00 -> 60.8 mm, vias 0 -> 1
- net KEY0: track 43.6 -> 0.00 mm, vias 2 -> 0
- net +5V: track 92.4 -> 135.7 mm
- net KEY5: track 0.00 -> 41.6 mm, vias 0 -> 1
- net KEY1: track 41.6 -> 76.6 mm, vias 2 -> 1
- net KEY2: track 69.6 -> 38.1 mm, vias 0 -> 1
- net N$4: track 28.2 -> 0.00 mm
- net TX: track 49.7 -> 23.7 mm, vias 1 -> 0
- net N$6: track 21.1 -> 0.00 mm
- net N$3: track 18.5 -> 0.00 mm
- net N$5: track 20.4 -> 37.1 mm, vias 0 -> 1
- net N$2: track 21.3 -> 4.84 mm
- net VPP: track 0.00 -> 14.0 mm, vias 0 -> 2
- net PGD: track 0.00 -> 13.4 mm, vias 0 -> 2
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Other:
- board text added: "MIDIWALL v3"
- board text removed: "MIDIWALL v2"

Commit message: ewr
Parts:
- removed LED1, LED2: (no value), led:LED3MM
- removed R10, R11, R4, R6, R7, R8, R9: (no value), rcl:R0805
- removed R5: 4k7, rcl:R0805
- added D2, D3: (no value), led:LED3MM
- C1: device rcl:E2,5-5 -> resistor:SMC_B
- D1: value 0805DIODE -> MBR0520LT; device jasons_stuff:0805DIODE -> diode:SOD123
- R3: value (none) -> 4k7
- moved R1 50.3 mm to (50.8, 26.7)
- moved R3 50.2 mm to (54.6, 30.9), turned to 0 degrees
- moved R2 46.1 mm to (50.8, 21.6)
- moved OUT 39.6 mm to (45.7, 40.6), turned to 0 degrees
- moved IN 39.1 mm to (35.6, 40.6), turned to 0 degrees
- moved C1 35.9 mm to (16.5, 35.6)
- moved D1 33.9 mm to (19.7, 35.6), turned to 90 degrees
- moved ICSP 17.3 mm to (64.0, 39.9), flipped to the bottom
- moved C2 8.52 mm to (62.4, 30.0)
- moved IC1 8.52 mm to (62.2, 24.1)
- moved SW1 1.80 mm to (22.9, 24.1)
- moved SW2 1.27 mm to (40.6, 24.1)
- moved SW3 1.27 mm to (22.9, 10.2), turned to 180 degrees
- moved SW5 1.27 mm to (58.4, 10.2), turned to 180 degrees
- turned SW4 to 180 degrees
Connections:
- removed net N$5: OUT.3, R11.1, R8.2
- removed net N$7: IN.2, IN.2A, R1.2, R4.1
- removed net N$8: OUT.2, OUT.2A, R10.1, R9.2
- removed net N$9: IN.3, R2.2, R3.1
- net +5V: now also D1.C, IN.2, IN.2A, OUT.2, OUT.2A; no longer D1.A, R10.2, R11.2, R4.2, R5.2
- net GND: now also D1.A, R1.1, R2.1; no longer D1.C, LED1.K, LED2.K
- net KEY1: now also IC1.10; no longer IC1.9
- net KEY3: now also IC1.9; no longer IC1.11
- net KEY4: now also IC1.11; no longer IC1.8
- net KEY5: now also IC1.8; no longer IC1.10
- net LED1: now also D2.A; no longer R6.2
- net LED2: now also D3.A; no longer R7.2
- net N$1: now also D2.K, R1.2; no longer LED1.A, R6.1
- net N$2: now also D3.K, R2.2; no longer LED2.A, R7.1
- net RX: now also IN.3, R3.1; no longer R1.1, R2.1, R5.1
- net TX: now also OUT.3; no longer R8.1, R9.1
Routing:
- net +5V: track 135.7 -> 71.8 mm, vias 2 -> 1
- net RX: track 93.2 -> 31.0 mm
- net N$5: track 37.1 -> 0.00 mm, vias 1 -> 0
- net N$7: track 29.3 -> 0.00 mm, vias 1 -> 0
- net KEY3: track 60.8 -> 35.6 mm, vias 1 -> 0
- net KEY1: track 76.6 -> 53.9 mm, vias 1 -> 0
- net KEY5: track 41.6 -> 20.2 mm, vias 1 -> 0
- net N$8: track 19.0 -> 0.00 mm
- net N$9: track 18.9 -> 0.00 mm, vias 1 -> 0
- net VPP: track 14.0 -> 24.7 mm, vias 2 -> 1
- net KEY4: track 64.1 -> 54.3 mm, vias 1 -> 0
- net PGC: track 6.41 -> 15.6 mm, vias 0 -> 1
- net PGD: track 13.4 -> 20.0 mm, vias 2 -> 1
- net KEY2: track 38.1 -> 32.5 mm, vias 1 -> 0
- net N$1: track 8.31 -> 3.94 mm
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Other:
- board size 80.7 x 36.8 mm -> 63.5 x 40.6 mm
- board text removed: "MIDIWALL v3"
- board text removed: "hotchk155"

Commit message: Version 4 PCB PROD
Parts:
- removed D1: MBR0520LT, diode:SOD123
- R1: value (none) -> 4k7
- R3: value 4k7 -> (none)
- moved R1 32.0 mm to (19.7, 34.3), turned to 90 degrees
- moved R3 10.0 mm to (50.8, 21.6), turned to 270 degrees
- moved R2 5.08 mm to (50.8, 26.7)
- moved C1 1.27 mm to (16.5, 34.3), turned to 270 degrees
Connections:
- net +5V: now also IN.3, OUT.3, R1.2; no longer D1.C, IN.2, IN.2A, OUT.2, OUT.2A, R3.2
- net GND: now also R3.1; no longer D1.A, R1.1
- net N$1: now also R2.2; no longer R1.2
- net N$2: now also R3.2; no longer R2.2
- net RX: now also IN.2, IN.2A, R1.1; no longer IN.3, R3.1
- net TX: now also OUT.2, OUT.2A; no longer OUT.3
Routing:
- net RX: track 31.0 -> 65.9 mm
- net TX: track 20.7 -> 33.2 mm
- net +5V: track 71.8 -> 66.7 mm
Other:
- board text added: "MIDIWALL V4"
- board text added: "hotchk155/2022"

Commit message: assdadasadsaddas
Parts:
- removed IC1: PIC16F1825SO14, jasons_stuff:SO14
- removed SW1, SW2, SW3, SW4, SW5: (no value), switch-omron:B3F-40XX
- added R4: (no value), rcl:R0805
- added U$1: PIC16F15345, jason_eagle6:TSSOP20
- added U$2, U$3, U$4, U$5, U$6: 6MMTACTSMT, jason_eagle6:6MMTACTSMT
- D2, D3: device led:LED3MM -> adafruit:CHIPLED_0805
- IN, OUT: value 3_5MM_PTH_MICRO -> 1503_02; device jason_eagle6:3_5MM_PTH_MICRO -> con-lumberg:1503_02
- moved ICSP 44.4 mm to (25.9, 17.0), flipped to the top
- moved C2 41.9 mm to (21.1, 22.9), turned to 270 degrees
- moved D2 31.5 mm to (30.5, 47.0)
- moved R2 30.6 mm to (22.9, 39.1)
- moved R3 30.0 mm to (21.1, 17.8), turned to 90 degrees
- moved D3 24.3 mm to (30.5, 19.1)
- moved OUT 16.0 mm to (36.8, 27.3), turned to 270 degrees
- moved R1 12.3 mm to (31.9, 33.0), turned to 270 degrees
- moved C1 6.48 mm to (22.9, 33.0)
- moved IN 2.29 mm to (36.8, 38.7), turned to 270 degrees
Connections:
- new net N$3: OUT.3, R4.1
- net +5V: now also R4.2, U$1.1; no longer IC1.1, OUT.3
- net GND: now also D2.C, D3.C, U$1.20, U$2.2, U$2.3, U$3.2, U$3.3, U$4.2, U$4.3, U$5.2, U$5.3, U$6.2, U$6.3; no longer IC1.14, R2.1, R3.1, SW1.1, SW1.2, SW2.1, SW2.2, SW3.1, SW3.2, SW4.1, SW4.2, SW5.1, SW5.2
- net KEY1: now also U$1.3, U$6.1, U$6.4; no longer IC1.10, SW3.3, SW3.4
- net KEY2: now also U$1.7, U$5.1, U$5.4; no longer IC1.7, SW2.3, SW2.4
- net KEY3: now also U$1.8, U$4.1, U$4.4; no longer IC1.9, SW4.3, SW4.4
- net KEY4: now also U$1.9, U$3.1, U$3.4; no longer IC1.11, SW1.3, SW1.4
- net KEY5: now also U$1.10, U$2.1, U$2.4; no longer IC1.8, SW5.3, SW5.4
- net LED1: now also R2.2, U$1.2; no longer D2.A, IC1.2
- net LED2: now also R3.2, U$1.16; no longer D3.A, IC1.3
- net N$1: now also D2.A, R2.1; no longer D2.K, R2.2
- net N$2: now also D3.A, R3.1; no longer D3.K, R3.2
- net PGC: now also U$1.18; no longer IC1.12
- net PGD: now also U$1.19; no longer IC1.13
- net RX: now also U$1.5; no longer IC1.5, IN.2A
- net TX: now also U$1.6; no longer IC1.6, OUT.2A
- net VPP: now also U$1.4; no longer IC1.4
Routing:
- net KEY1: track 53.9 -> 14.9 mm
- net KEY4: track 54.3 -> 15.4 mm
- net RX: track 65.9 -> 37.0 mm
- net +5V: track 66.7 -> 50.4 mm, vias 1 -> 0
- net LED1: track 5.55 -> 20.9 mm
- net VPP: track 24.7 -> 12.6 mm, vias 1 -> 2
- net N$3: track 0.00 -> 9.76 mm
- net KEY5: track 20.2 -> 11.3 mm
- net N$1: track 3.94 -> 12.0 mm
- net KEY3: track 35.6 -> 28.4 mm
- net TX: track 33.2 -> 26.7 mm, vias 1 -> 2
- net PGD: track 20.0 -> 13.5 mm, vias 1 -> 2
- net N$2: track 3.94 -> 9.27 mm
- net PGC: track 15.6 -> 10.8 mm, vias 1 -> 0
- net KEY2: track 32.5 -> 28.4 mm
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Other:
- board size 63.5 x 40.6 mm -> 36.8 x 45.6 mm
- board text removed: "MIDIWALL V4"
- board text removed: "hotchk155/2022"
