File: hardware/midiwall.sch (EAGLE design)
At the start: 29 parts, among them IC1 PIC12F1822SO08

Commit message: new case
Parts:
- R5: value (none) -> 4k7
Other:
- note added: "R4/R1, R7/R10 - MMA R3/R2, R8/R9 - NOVATION/ARTURIA"
Changed lines of the file:
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@@
 <part name="R10" library="rcl" deviceset="R-EU_" device="R0805"/>
 <part name="P+2" library="supply1" deviceset="+5V" device=""/>
-<part name="R5" library="rcl" deviceset="R-EU_" device="R0805"/>
+<part name="R5" library="rcl" deviceset="R-EU_" device="R0805" value="4k7"/>
 <part name="P+3" library="supply1" deviceset="+5V" device=""/>
 <part name="P+4" library="supply1" deviceset="+5V" device=""/>
@@
 <sheet>
 <plain>
+<text x="5.08" y="185.42" size="1.778" layer="97">R4/R1, R7/R10 - MMA
+R3/R2, R8/R9 - NOVATION/ARTURIA</text>
 </plain>
 <instances>
@@
 <instance part="GND2" gate="1" x="15.24" y="78.74"/>
 <instance part="GND3" gate="1" x="22.86" y="78.74"/>
-<instance part="R1" gate="G$1" x="0" y="142.24" rot="R90"/>
-<instance part="R2" gate="G$1" x="2.54" y="142.24" rot="R90"/>
+<instance part="R1" gate="G$1" x="0" y="142.24" smashed="yes" rot="R90">
+<attribute name="NAME" x="-1.4986" y="138.43" size="1.778" layer="95" rot="R90"/>
+<attribute name="VALUE" x="3.302" y="138.43" size="1.778" layer="96" rot="R90"/>
+</instance>
+<instance part="R2" gate="G$1" x="2.54" y="142.24" smashed="yes" rot="R90">
+<attribute name="NAME" x="6.1214" y="138.43" size="1.778" layer="95" rot="R90"/>
+<attribute name="VALUE" x="5.842" y="138.43" size="1.778" layer="96" rot="R90"/>
+</instance>
 <instance part="GND4" gate="1" x="15.24" y="134.62"/>
-<instance part="R8" gate="G$1" x="30.48" y="165.1" rot="R90"/>
+<instance part="R8" gate="G$1" x="30.48" y="165.1" smashed="yes" rot="R90">
+<attribute name="NAME" x="34.0614" y="161.29" size="1.778" layer="95" rot="R90"/>
+<attribute name="VALUE" x="33.782" y="161.29" size="1.778" layer="96" rot="R90"/>
+</instance>
 <instance part="P+1" gate="1" x="30.48" y="180.34"/>
-<instance part="R4" gate="G$1" x="2.54" y="165.1" rot="R90"/>
-<instance part="R3" gate="G$1" x="0" y="165.1" rot="R90"/>
-<instance part="R7" gate="G$1" x="27.94" y="165.1" rot="R90"/>
-<instance part="R9" gate="G$1" x="27.94" y="142.24" rot="R90"/>
-<instance part="R10" gate="G$1" x="30.48" y="142.24" rot="R90"/>
+<instance part="R4" gate="G$1" x="2.54" y="165.1" smashed="yes" rot="R90">
+<attribute name="NAME" x="6.1214" y="163.83" size="1.778" layer="95" rot="R90"/>
+<attribute name="VALUE" x="5.842" y="161.29" size="1.778" layer="96" rot="R90"/>
+</instance>
+<instance part="R3" gate="G$1" x="0" y="165.1" smashed="yes" rot="R90">
+<attribute name="NAME" x="-1.4986" y="161.29" size="1.778" layer="95" rot="R90"/>
+<attribute name="VALUE" x="3.302" y="161.29" size="1.778" layer="96" rot="R90"/>
+</instance>
+<instance part="R7" gate="G$1" x="27.94" y="165.1" smashed="yes" rot="R90">
+<attribute name="NAME" x="26.4414" y="161.29" size="1.778" layer="95" rot="R90"/>
+<attribute name="VALUE" x="31.242" y="161.29" size="1.778" layer="96" rot="R90"/>
+</instance>
+<instance part="R9" gate="G$1" x="27.94" y="142.24" smashed="yes" rot="R90">
+<attribute name="NAME" x="26.4414" y="138.43" size="1.778" layer="95" rot="R90"/>
+<attribute name="VALUE" x="31.242" y="138.43" size="1.778" layer="96" rot="R90"/>
+</instance>
+<instance part="R10" gate="G$1" x="30.48" y="142.24" smashed="yes" rot="R90">
+<attribute name="NAME" x="34.0614" y="138.43" size="1.778" layer="95" rot="R90"/>
+<attribute name="VALUE" x="33.782" y="138.43" size="1.778" layer="96" rot="R90"/>
+</instance>
 <instance part="P+2" gate="1" x="0" y="180.34"/>
-<instance part="R5" gate="G$1" x="7.62" y="142.24" rot="R90"/>
+<instance part="R5" gate="G$1" x="7.62" y="142.24" smashed="yes" rot="R90">
+<attribute name="NAME" x="11.2014" y="143.51" size="1.778" layer="95" rot="R90"/>
+<attribute name="VALUE" x="10.922" y="138.43" size="1.778" layer="96" rot="R90"/>
+</instance>
 <instance part="P+3" gate="1" x="7.62" y="152.4"/>
 <instance part="P+4" gate="1" x="15.24" y="124.46"/>
@@
 </schematic>
 </drawing>
+<compatibility>
+<note version="6.3" minversion="6.2.2" severity="warning">
+Since Version 6.2.2 text objects can contain more than one line,
+which will not be processed correctly with this version.
+</note>
+</compatibility>
 </eagle>

Commit message: REV3
Parts:
- removed D2, D3, D4, D5, D6, D7: 0805DIODE, jasons_stuff:0805DIODE
- removed J1: (no value), tag-connect:TC2030-MCP-NL
- added ICSP: (no value), tag-connect:TC2030-MCP-NL
- added LED2: (no value), led:LED3MM
- added R11: (no value), rcl:R-EU_R0805
- C1: device microbuilder:CAP_TANTALUMA/3216_REFLOW -> rcl:CPOL-EUE2.5-5
- IC1: value PIC12F1822SO08 -> PIC16F1825SO14; device jasons_stuff:PIC12F1822SO08 -> jasons_stuff:PIC16F1825SO14
Connections:
- removed net KEY0: D5.P$1, D6.P$1, IC1.MCLR#/VPP/RA3, J1.VPP/MCLR
- removed net N$10: LED1.C, R6.2
- removed net N$11: IC1.RA5, LED1.A
- removed net N$3: D7.P$2, SW4.P, SW4.P1
- removed net N$4: D1.P$2, D5.P$2, SW2.P, SW2.P1
- removed net N$6: D3.P$2, D4.P$2, SW3.P, SW3.P1
- new net KEY3: IC1.RA2/INT, SW4.P, SW4.P1
- new net KEY4: IC1.RC2, SW1.P, SW1.P1
- new net KEY5: IC1.RCO/SCL/SCK, SW5.P, SW5.P1
- new net LED1: IC1.RA5, R6.2
- new net LED2: IC1.RA4/SDO, R7.2
- new net PGC: IC1.RA1/ICPCLK, ICSP.ICSP_CLK/PGC
- new net PGD: IC1.RA0/ICSPDAT, ICSP.ICSP_DAT/PGD
- new net VPP: IC1.RA3/MCLR#/VPP, ICSP.VPP/MCLR
- net +5V: now also D1.P$2, ICSP.VDD, R10.2, R11.2; no longer J1.VDD, R7.2, R8.2
- net GND: now also D1.P$1, ICSP.VSS(GND), LED1.C, LED2.C; no longer J1.VSS(GND), R6.1
- net KEY1: now also IC1.RC1/SDA/SDI, SW3.P, SW3.P1; no longer D1.P$1, D2.P$1, D3.P$1, IC1.RA4
- net KEY2: now also IC1.RC3/SS#, SW2.P, SW2.P1; no longer D4.P$1, D7.P$1, IC1.RA2
- net N$1: now also LED1.A, R6.1; no longer D6.P$2, SW5.P, SW5.P1
- net N$2: now also LED2.A, R7.1; no longer D2.P$2, SW1.P, SW1.P1
- net N$5: now also R11.1, R8.2; no longer R7.1, R9.2
- net N$7: now also R4.1; no longer R3.1
- net N$8: now also R10.1, R9.2; no longer R10.2, R8.1
- net N$9: now also R3.1; no longer R4.1
- net RX: now also IC1.RC5/RX; no longer IC1.RA1/PGC, J1.ICSP_CLK/PGC
- net TX: now also IC1.RC4/TX, R8.1; no longer IC1.RA0/PGD, J1.ICSP_DAT/PGD, R10.1
Other:
- note added: "CC-NC-BY-SA"
- note added: "MIDIWALL rev 3"
- note added: "October 2019 - Sixty four pixels ltd"
- note removed: "R4/R1, R7/R10 - MMA R3/R2, R8/R9 - NOVATION/ARTURIA"
- moved on the sheet: C2, D1, LED1, R10, R3, R4, R6, R7, R8, R9, SW1, SW2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

Commit message: ewr
Parts:
- removed R10, R11, R4, R6, R7, R8, R9: (no value), rcl:R-EU_R0805
- removed R5: 4k7, rcl:R-EU_R0805
- C1: device rcl:CPOL-EUE2.5-5 -> resistor:CPOL-EUSMCB
- D1: value 0805DIODE -> MBR0520LT; device jasons_stuff:0805DIODE -> diode:MBR0520LT
- R3: value (none) -> 4k7
- renumbered LED1 to D2, LED2 to D3
Connections:
- removed net N$5: OUT.3, R11.1, R8.2
- removed net N$7: IN.4, R1.2, R4.1
- removed net N$8: OUT.4, R10.1, R9.2
- removed net N$9: IN.3, R2.2, R3.1
- net +5V: now also D1.C, IN.4, OUT.4; no longer D1.P$2, R10.2, R11.2, R4.2, R5.2
- net GND: now also D1.A, R1.1, R2.1; no longer D1.P$1, D2.C, D3.C
- net KEY1: now also IC1.RCO/SCL/SCK; no longer IC1.RC1/SDA/SDI
- net KEY3: now also IC1.RC1/SDA/SDI; no longer IC1.RA2/INT
- net KEY4: now also IC1.RA2/INT; no longer IC1.RC2
- net KEY5: now also IC1.RC2; no longer IC1.RCO/SCL/SCK
- net LED1: now also D2.A; no longer R6.2
- net LED2: now also D3.A; no longer R7.2
- net N$1: now also D2.C, R1.2; no longer D2.A, R6.1
- net N$2: now also D3.C, R2.2; no longer D3.A, R7.1
- net RX: now also IN.3, R3.1; no longer R1.1, R2.1, R5.1
- net TX: now also OUT.3; no longer R8.1, R9.1
Other:
- moved on the sheet: R1, R2, R3

Commit message: Version 4 PCB PROD
Parts:
- removed D1: MBR0520LT, diode:MBR0520LT
- R1: value (none) -> 4k7
- R3: value 4k7 -> (none)
Connections:
- net +5V: now also IN.3, OUT.3, R1.2; no longer D1.C, IN.4, OUT.4, R3.2
- net GND: now also R3.1; no longer D1.A, R1.1
- net N$1: now also R2.2; no longer R1.2
- net N$2: now also R3.2; no longer R2.2
- net RX: now also IN.4, R1.1; no longer IN.3, R3.1
- net TX: now also OUT.4; no longer OUT.3
Other:
- note added: "Jan 2022 - Sixty four pixels ltd"
- note added: "MIDIWALL rev 4"
- note removed: "MIDIWALL rev 3"
- note removed: "October 2019 - Sixty four pixels ltd"
- moved on the sheet: IN, OUT, R1, R2, R3

Commit message: assdadasadsaddas
Parts:
- removed IC1: PIC16F1825SO14, jasons_stuff:PIC16F1825SO14
- removed SW1, SW2, SW3, SW4, SW5: (no value), switch-omron:40-XX
- added R4: (no value), rcl:R-EU_R0805
- added U$1: PIC16F15345, jason_eagle6:PIC16F15345
- added U$2, U$3, U$4, U$5, U$6: 6MMTACTSMT, jason_eagle6:6MMTACTSMT
- D2, D3: device led:LED3MM -> adafruit:LEDCHIPLED_0805
- IN, OUT: value 3_5MM_PTH_MICRO -> 1503_02; device jason_eagle6:3_5MM_PTH_MICRO -> con-lumberg:1503_02
Connections:
- new net N$3: OUT.3, R4.1
- net +5V: now also R4.2, U$1.VDD; no longer IC1.VDD, OUT.3
- net GND: now also D2.C, D3.C, IN.1, OUT.1, U$1.VSS, U$2.2, U$2.3, U$3.2, U$3.3, U$4.2, U$4.3, U$5.2, U$5.3, U$6.2, U$6.3; no longer IC1.VSS, IN.2, OUT.2, R2.1, R3.1, SW1.S, SW1.S1, SW2.S, SW2.S1, SW3.S, SW3.S1, SW4.S, SW4.S1, SW5.S, SW5.S1
- net KEY1: now also U$1.RA4, U$6.1, U$6.4; no longer IC1.RCO/SCL/SCK, SW3.P, SW3.P1
- net KEY2: now also U$1.RC3, U$5.1, U$5.4; no longer IC1.RC3/SS#, SW2.P, SW2.P1
- net KEY3: now also U$1.RC6, U$4.1, U$4.4; no longer IC1.RC1/SDA/SDI, SW4.P, SW4.P1
- net KEY4: now also U$1.RC7, U$3.1, U$3.4; no longer IC1.RA2/INT, SW1.P, SW1.P1
- net KEY5: now also U$1.RB7, U$2.1, U$2.4; no longer IC1.RC2, SW5.P, SW5.P1
- net LED1: now also R2.2, U$1.RA5; no longer D2.A, IC1.RA5
- net LED2: now also R3.2, U$1.RC0; no longer D3.A, IC1.RA4/SDO
- net N$1: now also D2.A, R2.1; no longer D2.C, R2.2
- net N$2: now also D3.A, R3.1; no longer D3.C, R3.2
- net PGC: now also U$1.RA1/PGC; no longer IC1.RA1/ICPCLK
- net PGD: now also U$1.RA0/PCD; no longer IC1.RA0/ICSPDAT
- net RX: now also IN.2, U$1.RC5; no longer IC1.RC5/RX, IN.4
- net TX: now also OUT.2, U$1.RC4; no longer IC1.RC4/TX, OUT.4
- net VPP: now also U$1.RA3/MCLR#; no longer IC1.RA3/MCLR#/VPP
Other:
- moved on the sheet: D2, D3, R2, R3
