File: hardware/midi_nubbin.sch (EAGLE design)
At the start: 17 parts

Commit message: MN V1 PCB?
Parts:
- removed D3: (no value), adafruit:LEDCHIPLED_0805
- added D1: (no value), adafruit:LEDCHIPLED_0805
- R1: value 4k7 -> (none)
- R2: value (none) -> 4k7
- renumbered U$1 to IC1, U$2 to SW5, U$3 to SW45, U$4 to SW3, U$5 to SW1, U$6 to SW2
Connections:
- net +5V: now also R2.2, R3.2; no longer R1.2, R4.2
- net GND: now also D1.C; no longer D3.C
- net LED1: now also R1.2; no longer R2.2
- net LED2: now also R4.2; no longer R3.2
- net N$1: now also D1.A, R1.1; no longer D2.A, R2.1
- net N$2: now also D2.A, R4.1; no longer D3.A, R3.1
- net N$3: now also R3.1; no longer R4.1
- net RX: now also R2.1; no longer R1.1
Other:
- note added: "Apr 2022 - Sixty four pixels ltd"
- note added: "MIDI NUBBIN rev 1"
- note added: "Ring (+5V)"
- note added: "Sleeve (GND)"
- note added: "Tip (Signal)"
- note removed: "Jan 2022 - Sixty four pixels ltd"
- note removed: "MIDIWALL rev 4"
- moved on the sheet: D2, R1, R2, R3, R4
