File: fascia/midi_nubbin_fascia/midi_nubbin_fascia.kicad_pcb (KiCad board)
At the start: 2 copper layers, 48.4 x 40.1 mm, 0 parts

Commit message: add generic fasica
Parts:
- added G***: LOGO, Library:generic-silk, F.Cu at (72.5, 70.3)
Other:
- board size 48.4 x 40.1 mm -> 74.4 x 116.4 mm
