File: fascia/midi_nubbin_fascia/midi_nubbin_fascia.kicad_pcb (KiCad board)
At the start: 2 copper layers, 48.4 x 40.1 mm, 1 part

Commit message: sd
Parts:
- moved G*** 79.6 mm to (148.5, 46.5)
Other:
- outline, holes or cut-outs redrawn
